Commit message: add IMU sensor

File: urdf/ausrabot.urdf.xacro (robot description, xacro)
@@ -333,4 +333,39 @@
       xyz="0 0 0" />
   </joint>
+  <link name="imu_link">
+    <visual>
+      <geometry>
+        <box size="0.0001 0.0001 0.0001"/>
+      </geometry>
+      <material name="">
+        <color rgba="1.0 0.0 0.0 1"/> </material>
+    </visual>
+    <collision>
+      <geometry>
+        <box size="0.0001 0.0001 0.0001"/>
+      </geometry>
+    </collision>
+    <inertial>
+      <mass value="0.01"/>
+      <inertia ixx="0.0001" ixy="0" ixz="0" iyy="0.0001" iyz="0" izz="0.0001"/>
+    </inertial>
+  </link>
+  <joint name="imu_joint" type="fixed">
+    <parent link="base_link"/>
+    <child link="imu_link"/>
+    <origin xyz="0 0 0" rpy="0 0 0"/>
+  </joint>
+  <gazebo reference="imu_link">
+    <sensor name="imu_sensor" type="imu">
+      <always_on>true</always_on>
+      <update_rate>100</update_rate>
+      <visualize>true</visualize>
+      <topic>imu</topic>
+      <plugin filename="libignition-gazebo-imu-system.so" name="ignition::gazebo::systems::Imu">
+      </plugin>
+      <pose>0 0 0 0 0 0</pose>
+      <gz_frame_id>imu_link</gz_frame_id>
+    </sensor>
+  </gazebo>
   <ros2_control name="GazeboSystem" type="system">
     <hardware>

Commit message: update-urdf-config-launch-to-match-cppDriver

File: urdf/ausrabot.urdf.xacro (robot description, xacro)
@@ -5,5 +5,5 @@
       <parent link="robot_footprint"/>
       <child link="base_link"/>
-      <origin xyz="0 0 0" rpy="0 0 0"/>
+      <origin xyz="0 0 0" rpy="0 0 -1.558930266"/>
   </joint>
   <link

Commit message: added camera plugin

File: urdf/ausrabot.urdf.xacro (robot description, xacro)
@@ -333,4 +333,10 @@
       xyz="0 0 0" />
   </joint>
+  <link name="camera_link_optical"/>
+  <joint name="camera_optical_joint" type="fixed">
+    <parent link="oak_camera"/>
+    <child link="camera_link_optical"/>
+    <origin xyz="0 0 -2" rpy="0 3.14 0"/>
+  </joint>
   <link name="imu_link">
     <visual>
@@ -356,16 +362,4 @@
     <origin xyz="0 0 0" rpy="0 0 0"/>
   </joint>
-  <gazebo reference="imu_link">
-    <sensor name="imu_sensor" type="imu">
-      <always_on>true</always_on>
-      <update_rate>100</update_rate>
-      <visualize>true</visualize>
-      <topic>imu</topic>
-      <plugin filename="libignition-gazebo-imu-system.so" name="ignition::gazebo::systems::Imu">
-      </plugin>
-      <pose>0 0 0 0 0 0</pose>
-      <gz_frame_id>imu_link</gz_frame_id>
-    </sensor>
-  </gazebo>
   <ros2_control name="GazeboSystem" type="system">
     <hardware>
@@ -447,3 +441,41 @@
       <gz_frame_id>lidar</gz_frame_id> </sensor>
   </gazebo>
+  <gazebo reference="imu_link">
+    <sensor name="imu_sensor" type="imu">
+      <always_on>true</always_on>
+      <update_rate>100</update_rate>
+      <visualize>true</visualize>
+      <topic>imu</topic>
+      <plugin filename="libignition-gazebo-imu-system.so" name="ignition::gazebo::systems::Imu">
+      </plugin>
+      <pose>0 0 0 0 0 0</pose>
+      <gz_frame_id>imu_link</gz_frame_id>
+    </sensor>
+  </gazebo>
+  <gazebo reference="oak_camera">
+    <sensor name="oak_d_lite_rgb" type="camera">
+      <pose>0 0 0 0 0 0</pose>
+      <visualize>true</visualize>
+      <update_rate>30.0</update_rate>
+      <topic>camera/image_raw</topic>
+      <gz_frame_id>camera_link_optical</gz_frame_id>
+      <camera>
+        <horizontal_fov>1.20428</horizontal_fov>
+        <image>
+          <width>1920</width>
+          <height>1080</height>
+          <format>R8G8B8</format>
+        </image>
+        <clip>
+          <near>0.08</near>
+          <far>100.0</far>
+        </clip>
+        <noise>
+          <type>gaussian</type>
+          <mean>0.0</mean>
+          <stddev>0.007</stddev>
+        </noise>
+      </camera>
+    </sensor>
+  </gazebo>
 </robot>
