Commit message: RGB-D camera fixes and urdf frame fixes

File: urdf/ausrabot/gazebo.xacro (robot description, xacro)
@@ -2,7 +2,5 @@
 <robot xmlns:xacro="http://www.ros.org/wiki/xacro">
   <xacro:macro name="gazebo">
-    <!-- ================================= -->
-    <!--       ROS2 CONTROL SYSTEM         -->
-    <!-- ================================= -->
+    <!-- ROS2 CONTROL -->
     <ros2_control name="GazeboSystem" type="system">
       <hardware>
@@ -25,7 +23,5 @@
       </joint>
     </ros2_control>
-    <!-- ================================= -->
-    <!--       GLOBAL GAZEBO PLUGINS       -->
-    <!-- ================================= -->
+    <!-- GAZEBO PLUGINS -->
     <gazebo>
       <plugin filename="gz-sim-sensors-system" name="gz::sim::systems::Sensors">
@@ -38,7 +34,5 @@
       </plugin>
     </gazebo>
-    <!-- ================================= -->
-    <!--         WHEEL FRICTION            -->
-    <!-- ================================= -->
+    <!-- WHEEL FRICTION -->
     <gazebo reference="wheel_1">
       <mu1>1.0</mu1>
@@ -56,11 +50,9 @@
       <fdir1>1 0 0</fdir1>
     </gazebo>
-    <!-- ================================= -->
-    <!--         SENSOR PLUGINS            -->
-    <!-- ================================= -->
+    <!-- SENSOR PLUGINS -->
     <!-- LiDAR Plugin -->
     <gazebo reference="lidar">
       <sensor name="lidar" type="gpu_lidar">
-        <pose relative_to='lidar'>0 0 0 0 0 0</pose>
+        <pose>0 0 0 0 0 ${pi}</pose>
         <topic>scan</topic>
         <update_rate>10</update_rate>
@@ -103,14 +95,27 @@
       </sensor>
     </gazebo>
-    <!-- Camera Plugin -->
+    <!-- RGBD Camera Plugin (Oak-D Lite) -->
+    <!-- CORRECTED: Changed pose from "0 0 0 0 -${pi/2} 0" to "0 0 0 0 0 0" -->
+    <!-- Gazebo camera sensors look along +X axis, which now correctly aligns with oak_camera +X (forward) -->
     <gazebo reference="oak_camera">
-      <sensor name="oak_d_lite_rgb" type="camera">
-        <pose>0 0 0 0 0 0</pose>
+      <sensor name="oak_d_lite_rgbd" type="rgbd_camera">
+        <pose>0 0 0 0 -${pi/2} 0</pose>
+        <always_on>true</always_on>
+        <update_rate>30.0</update_rate>
         <visualize>true</visualize>
-        <update_rate>30.0</update_rate>
-        <topic>camera/image_raw</topic>
+        <topic>rgbd_camera</topic>
+        <!-- Frame ID sets the Header.stamp in ROS. Matches the Optical Frame TF -->
         <gz_frame_id>camera_link_optical</gz_frame_id>
-        <camera>
+        <camera name="oak_d_lite">
           <horizontal_fov>1.20428</horizontal_fov>
+          <lens>
+            <intrinsics>
+              <fx>1382.0</fx>
+              <fy>1382.0</fy>
+              <cx>960.0</cx>
+              <cy>540.0</cy>
+              <s>0</s>
+            </intrinsics>
+          </lens>
           <image>
             <width>1920</width>
@@ -122,4 +127,10 @@
             <far>100.0</far>
           </clip>
+          <depth_camera>
+            <clip>
+              <near>0.1</near>
+              <far>10.0</far>
+            </clip>
+          </depth_camera>
           <noise>
             <type>gaussian</type>

File: urdf/ausrabot/sensors.xacro (robot description, xacro)
@@ -27,9 +27,9 @@
     </link>
     <joint name="lidar_joint" type="fixed">
-      <origin xyz="-2.85102614102555E-05 0 0.130598095199185" rpy="0 0 3.14159265358979" />
+      <origin xyz="-2.85102614102555E-05 0 0.130598095199185" rpy="0 0 0" />
       <parent link="base_link" />
       <child link="lidar" />
     </joint>
-    <!-- OAK Camera Physical -->
+    <!-- OAK Camera Physical (from CAD) -->
     <link name="oak_camera">
       <inertial>
@@ -56,14 +56,26 @@
     </link>
     <joint name="oak_joint" type="fixed">
-      <origin xyz="0.000808669644363073 0.103689225067774 0.098888095199185" rpy="1.55867308825253 -1.5707963267949 0" />
+      <!-- CORRECTED: Changed from rpy="0 ${pi/2} ${pi/2}" to rpy="0 0 ${pi/2}" -->
+      <!-- This rotates oak_camera so its +X axis points in base_link +Y direction (forward) -->
+      <origin xyz="0.000808669644363073 0.103689225067774 0.098888095199185" rpy="0 ${pi/2} ${pi/2}" />
       <parent link="base_link" />
       <child link="oak_camera" />
     </joint>
-    <!-- Optical Link (Needed for TF) -->
+    <!-- Camera Link (standard ROS body frame: X forward, Y left, Z up) -->
+    <link name="camera_link"/>
+    <joint name="camera_link_joint" type="fixed">
+      <parent link="oak_camera"/>
+      <child link="camera_link"/>
+      <origin xyz="0 0 0" rpy="${pi/2} -${pi/2} -${pi/2}"/>
+    </joint>
+    <!-- Optical Frame (camera convention: Z forward/depth, X right, Y down) -->
+    <!-- CORRECTED: Standard ROS body-to-optical transformation -->
     <link name="camera_link_optical"/>
     <joint name="camera_optical_joint" type="fixed">
       <parent link="oak_camera"/>
       <child link="camera_link_optical"/>
-      <origin xyz="0 0 0" rpy="0 3.14 0"/>
+      <!-- Transform from oak_camera body frame (X=forward, Y=left, Z=up)
+           to optical frame (Z=forward, X=right, Y=down) -->
+      <origin xyz="0 0 0" rpy="${pi/2} ${pi/2} -${pi/2}"/>
     </joint>
     <!-- IMU Physical -->

File: urdf/ausrabot_full.urdf.xacro (robot description, xacro)
@@ -9,5 +9,5 @@
       <parent link="robot_footprint"/>
       <child link="base_link"/>
-      <origin xyz="0 0 0" rpy="0 0 0"/>
+      <origin xyz="0 0 0" rpy="0 0 ${pi}"/>
   </joint>
   <xacro:sensors />
