Commit message: fix-frames-in-URDF

File: urdf/ausrabot/ausrabot_core.xacro (robot description, xacro)
@@ -46,12 +46,4 @@
             <cylinder radius="0.034" length="0.015"/>
         </geometry>
-        <surface>
-          <friction>
-            <ode>
-              <mu>1.0</mu>
-              <mu2>1.0</mu2>
-            </ode>
-          </friction>
-        </surface>
       </collision>
     </link>
@@ -83,12 +75,4 @@
             <cylinder radius="0.034" length="0.015"/>
         </geometry>
-        <surface>
-          <friction>
-            <ode>
-              <mu>1.0</mu>
-              <mu2>1.0</mu2>
-            </ode>
-          </friction>
-        </surface>
       </collision>
     </link>
@@ -120,12 +104,4 @@
             <cylinder radius="0.034" length="0.015"/>
         </geometry>
-        <surface>
-          <friction>
-            <ode>
-              <mu>1.0</mu>
-              <mu2>1.0</mu2>
-            </ode>
-          </friction>
-        </surface>
       </collision>
     </link>

File: urdf/ausrabot/gazebo.xacro (robot description, xacro)
@@ -52,7 +52,8 @@
     <!-- SENSOR PLUGINS -->
     <!-- LiDAR Plugin -->
+    <!-- CORRECTED: Changed pose from "0 0 0 0 0 0" to "0 0 0 0 0 ${pi}" -->
     <gazebo reference="lidar">
       <sensor name="lidar" type="gpu_lidar">
-        <pose>0 0 0 0 0 ${pi}</pose>
+        <pose>0 0 0 0 0 0</pose>
         <topic>scan</topic>
         <update_rate>10</update_rate>

File: urdf/ausrabot/sensors.xacro (robot description, xacro)
@@ -27,5 +27,6 @@
     </link>
     <joint name="lidar_joint" type="fixed">
-      <origin xyz="-2.85102614102555E-05 0 0.130598095199185" rpy="0 0 0" />
+      <!-- LiDAR joint frame rotated by angle: 180 degrees (pi rad) -->
+      <origin xyz="-2.85102614102555E-05 0 0.130598095199185" rpy="0 0 ${pi}" />
       <parent link="base_link" />
       <child link="lidar" />
@@ -101,5 +102,6 @@
       <parent link="base_link"/>
       <child link="imu_link"/>
-      <origin xyz="0 0 0" rpy="0 0 0"/>
+      <!-- IMU joint frame rotated by angle: 90 degrees (pi/2 rad) -->
+      <origin xyz="0 0 0" rpy="0 0 ${pi/2}"/>
     </joint>
   </xacro:macro>

File: urdf/ausrabot_full.urdf.xacro (robot description, xacro)
@@ -9,5 +9,6 @@
       <parent link="robot_footprint"/>
       <child link="base_link"/>
-      <origin xyz="0 0 0" rpy="0 0 ${pi}"/>
+      <!-- Transformation between Gazebo world frame and the robot model's frame is -1.558930266 -->
+      <origin xyz="0 0 0" rpy="0 0 -1.558930266"/>
   </joint>
   <xacro:sensors />

Commit message: update meshes and xacro files and controller config params

File: urdf/ausrabot/ausrabot_core.xacro (robot description, xacro)
@@ -4,8 +4,9 @@
     <link name="base_link">
       <inertial>
-        <origin xyz="0.000132358596962433 0.0107784527153615 0.0455578201137751" rpy="0 0 0" />
-        <mass value="0.545316432015797" />
-        <inertia ixx="0.00232840648283892" ixy="7.82952052633134E-08" ixz="-2.35921291442106E-08"
-                 iyy="0.00246732309842302" iyz="-2.45394203695068E-06" izz="0.00451259615315152" />
+        <origin xyz="-0.00177767886836495 -7.08145711406941E-05 0.0345244109350669" rpy="0 0 0" />
+        <mass value="0.749591825708612" />
+        <inertia
+          ixx="0.00560242940522896" ixy="-3.10886247756778E-06" ixz="7.02379711896478E-05"
+          iyy="0.00543989398233584" iyz="-2.42126647279533E-17" izz="0.00951025265754031" />
       </inertial>
       <visual>
@@ -27,8 +28,9 @@
     <link name="wheel_1">
       <inertial>
-        <origin xyz="-6.11585138939009E-07 2.40519083084118E-06 0.00687917878282576" rpy="0 0 0" />
-        <mass value="0.037694823031467" />
-        <inertia ixx="3.0972076096957E-06" ixy="2.84246335131892E-11" ixz="-2.16478688549662E-10"
-                 iyy="3.09696234654175E-06" iyz="8.51072894756962E-10" izz="5.34864718246412E-06" />
+        <origin xyz="1.0863E-06 -2.2552E-06 0.0075339" rpy="0 0 0" />
+        <mass value="0.039266" />
+        <inertia
+          ixx="3.5298E-06" ixy="1.754E-10" ixz="1.4711E-10"
+          iyy="3.5298E-06" iyz="-1.6617E-10" izz="5.3943E-06" />
       </inertial>
       <visual>
@@ -44,5 +46,5 @@
         <origin xyz="0 0 0" rpy="0 0 0" />
         <geometry>
-            <cylinder radius="0.034" length="0.015"/>
+          <mesh filename="package://ausrabot_description/meshes/wheel_1.STL" />
         </geometry>
         <surface>
@@ -57,5 +59,5 @@
     </link>
     <joint name="joint_1" type="continuous">
-      <origin xyz="0.00131071109492098 0.110453635935089 -0.0161803398874989" rpy="1.5707963267949 0 3.12946941504743" />
+      <origin xyz="0.12368 -0.00013859 -0.019" rpy="1.5708 0 1.5708" />
       <parent link="base_link" />
       <child link="wheel_1" />
@@ -64,8 +66,9 @@
     <link name="wheel_2">
       <inertial>
-        <origin xyz="-2.22775634618061E-06 -1.09358984268573E-06 0.006879178822061" rpy="0 0 0" />
-        <mass value="0.0376948232954181" />
-        <inertia ixx="3.09702282374251E-06" ixy="-3.32677650778434E-11" ixz="-7.88279016321689E-10"
-                 iyy="3.09712667239217E-06" iyz="-3.87033927352786E-10" izz="5.34862673117426E-06" />
+        <origin xyz="1.0862E-06 -2.255E-06 0.0075339" rpy="0 0 0" />
+        <mass value="0.039266" />
+        <inertia
+          ixx="3.5297E-06" ixy="3.9609E-11" ixz="1.471E-10"
+          iyy="3.5297E-06" iyz="-1.6617E-10" izz="5.3942E-06" />
       </inertial>
       <visual>
@@ -75,5 +78,5 @@
         </geometry>
         <material name="">
-          <color rgba="0.0 0.0 1.0 1" />
+           <color rgba="0.0 0.0 1.0 1" />
         </material>
       </visual>
@@ -81,5 +84,5 @@
         <origin xyz="0 0 0" rpy="0 0 0" />
         <geometry>
-            <cylinder radius="0.034" length="0.015"/>
+          <mesh filename="package://ausrabot_description/meshes/wheel_2.STL" />
         </geometry>
         <surface>
@@ -94,5 +97,5 @@
     </link>
     <joint name="joint_2" type="continuous">
-      <origin xyz="-0.0963609169452294 -0.0540793874249231 -0.016180339887499" rpy="1.5707963267949 0 -1.05932078973896" />
+      <origin xyz="-0.062025 0.10707 -0.019" rpy="1.5708 0 -2.618" />
       <parent link="base_link" />
       <child link="wheel_2" />
@@ -101,8 +104,9 @@
     <link name="wheel_3">
       <inertial>
-        <origin xyz="2.39002105834052E-06 6.6831361357142E-07 0.00687917877739805" rpy="0 0 0" />
-        <mass value="0.0376948233023577" />
-        <inertia ixx="3.09710830531407E-06" ixy="8.8846112421192E-12" ixz="8.45711274919436E-10"
-                 iyy="3.0971477806935E-06" iyz="2.36549362165485E-10" izz="5.34873332719162E-06" />
+        <origin xyz="1.0862E-06 -2.2551E-06 0.0075339" rpy="0 0 0" />
+        <mass value="0.039266" />
+        <inertia
+          ixx="3.5297E-06" ixy="6.0263E-11" ixz="1.471E-10"
+          iyy="3.5296E-06" iyz="-1.6618E-10" izz="5.3941E-06" />
       </inertial>
       <visual>
@@ -112,5 +116,5 @@
         </geometry>
         <material name="">
-          <color rgba="0.0 0.0 1.0 1" />
+           <color rgba="0.0 0.0 1.0 1" />
         </material>
       </visual>
@@ -118,5 +122,5 @@
         <origin xyz="0 0 0" rpy="0 0 0" />
         <geometry>
-            <cylinder radius="0.034" length="0.015"/>
+          <mesh filename="package://ausrabot_description/meshes/wheel_3.STL" />
         </geometry>
         <surface>
@@ -131,5 +135,5 @@
     </link>
     <joint name="joint_3" type="continuous">
-      <origin xyz="0.0949646750660746 -0.0563989868566714 -0.016180339887499" rpy="1.5707963267949 0 1.03507431265423" />
+      <origin xyz="-0.062024 -0.10735 -0.019" rpy="1.5708 0 -0.5236" />
       <parent link="base_link" />
       <child link="wheel_3" />

File: urdf/ausrabot/gazebo.xacro (robot description, xacro)
@@ -54,5 +54,5 @@
     <gazebo reference="lidar">
       <sensor name="lidar" type="gpu_lidar">
-        <pose>0 0 0 0 0 ${pi}</pose>
+        <pose>0 0 0 0 0 0</pose>
         <topic>scan</topic>
         <update_rate>10</update_rate>

File: urdf/ausrabot/sensors.xacro (robot description, xacro)
@@ -5,8 +5,9 @@
     <link name="lidar">
       <inertial>
-        <origin xyz="-0.000173277491394453 -0.00676662791697095 0.00557928889827741" rpy="0 0 0" />
-        <mass value="0.171177012505295" />
-        <inertia ixx="0.000124253941113825" ixy="-4.38664000869312E-07" ixz="-6.40588163757229E-07"
-                 iyy="7.95393375273759E-05" iyz="-2.02744127539845E-05" izz="0.000141905084169328" />
+        <origin xyz="0.0067682 -0.00020713 -0.022521" rpy="0 0 0" />
+        <mass value="0.17118" />
+        <inertia
+          ixx="7.9535E-05" ixy="-1.035E-07" ixz="2.0281E-05"
+          iyy="0.00012426" iyz="-3.9476E-07" izz="0.00014191" />
       </inertial>
       <visual>
@@ -16,5 +17,5 @@
         </geometry>
         <material name="">
-          <color rgba="0.25 0.25 0.25 1" />
+          <color rgba="0.79216 0.81961 0.93333 1" />
         </material>
       </visual>
@@ -27,15 +28,16 @@
     </link>
     <joint name="lidar_joint" type="fixed">
-      <origin xyz="-2.85102614102555E-05 0 0.130598095199185" rpy="0 0 0" />
+      <origin xyz="-0.00012313 -2.5346E-05 0.1797" rpy="0 0 0" />
       <parent link="base_link" />
       <child link="lidar" />
+      <axis xyz="0 0 0" />
     </joint>
-    <!-- OAK Camera Physical (from CAD) -->
-    <link name="oak_camera">
+<link name="oak_camera">
       <inertial>
-        <origin xyz="2.77555756156289E-17 2.38524477946811E-18 -0.00860000000000001" rpy="0 0 0" />
-        <mass value="0.0417182941210436" />
-        <inertia ixx="2.88248605870479E-05" ixy="-7.46277402243113E-19" ixz="3.67148828118008E-22"
-                 iyy="3.55432167309084E-06" iyz="2.8124140826834E-22" izz="3.03221922380105E-05" />
+        <origin xyz="-0.0086 -5.8579E-18 0" rpy="0 0 0" />
+        <mass value="0.041718" />
+        <inertia
+          ixx="3.0322E-05" ixy="-8.0273E-23" ixz="-4.5515E-23"
+          iyy="3.5543E-06" iyz="-4.7563E-21" izz="2.8825E-05" />
       </inertial>
       <visual>
@@ -45,5 +47,5 @@
         </geometry>
         <material name="">
-          <color rgba="0.25 0.25 0.25 1" />
+          <color rgba="0.25098 0.25098 0.25098 1" />
         </material>
       </visual>
@@ -56,9 +58,8 @@
     </link>
     <joint name="oak_joint" type="fixed">
-      <!-- CORRECTED: Changed from rpy="0 ${pi/2} ${pi/2}" to rpy="0 0 ${pi/2}" -->
-      <!-- This rotates oak_camera so its +X axis points in base_link +Y direction (forward) -->
-      <origin xyz="0.000808669644363073 0.103689225067774 0.098888095199185" rpy="0 ${pi/2} ${pi/2}" />
+      <origin xyz="0.12008 -0.00013908 0.12046" rpy="0 0 0" />
       <parent link="base_link" />
       <child link="oak_camera" />
+      <axis xyz="0 0 0" />
     </joint>
     <!-- Camera Link (standard ROS body frame: X forward, Y left, Z up) -->
@@ -67,5 +68,5 @@
       <parent link="oak_camera"/>
       <child link="camera_link"/>
-      <origin xyz="0 0 0" rpy="${pi/2} -${pi/2} -${pi/2}"/>
+      <origin xyz="0 0 0" rpy="0 ${pi/2} 0"/>
     </joint>
     <!-- Optical Frame (camera convention: Z forward/depth, X right, Y down) -->
@@ -73,9 +74,9 @@
     <link name="camera_link_optical"/>
     <joint name="camera_optical_joint" type="fixed">
-      <parent link="oak_camera"/>
+      <parent link="camera_link"/>
       <child link="camera_link_optical"/>
       <!-- Transform from oak_camera body frame (X=forward, Y=left, Z=up)
            to optical frame (Z=forward, X=right, Y=down) -->
-      <origin xyz="0 0 0" rpy="${pi/2} ${pi/2} -${pi/2}"/>
+      <origin xyz="0 0 0" rpy="0 0 -${pi/2}"/>
     </joint>
     <!-- IMU Physical -->

File: urdf/ausrabot_full.urdf.xacro (robot description, xacro)
@@ -9,5 +9,5 @@
       <parent link="robot_footprint"/>
       <child link="base_link"/>
-      <origin xyz="0 0 0" rpy="0 0 ${pi}"/>
+      <origin xyz="0 0 0.05" rpy="0 0 0"/>
   </joint>
   <xacro:sensors />
